File: rp2350_dev_board.kicad_pcb (KiCad board)
At the start: 2 copper layers, 50 x 50 mm, 33 parts, among them J1 USB_B_Micro, J2 Conn_01x03_Socket, SW1 TS110426045, SW2 TS110426045, U1 RP2350A, U2 NCP1117-3.3_SOT223, U3 W25Q32JVSS, Y1 Crystal_GND24

Commit message: Minimal board complete
Parts:
- C2: value C -> 100n
- R2: value 2K -> 1k
- moved Y1 72.8 mm to (142.5, 109.1)
- moved SW2 60.8 mm to (155.2, 103.7)
- moved J2 58.9 mm to (157.7, 110.0), turned to -90 degrees
- moved R4 56.5 mm to (162.3, 106.4), turned to -90 degrees
- moved C3 52.3 mm to (140.4, 106.0)
- moved R2 51.5 mm to (144.0, 101.9), turned to 90 degrees
- moved C4 51.4 mm to (145.1, 106.0), turned to 180 degrees
- moved C16 49.0 mm to (150.5, 99.7), turned to 180 degrees
- moved C10 48.6 mm to (145.0, 101.9), turned to 90 degrees
- moved U3 47.1 mm to (135.2, 84.2)
- moved C18 45.0 mm to (142.6, 101.2), turned to 90 degrees
- moved C11 41.8 mm to (151.3, 94.6), turned to 180 degrees
- moved C9 40.5 mm to (149.5, 90.0), turned to -90 degrees
- moved C17 40.2 mm to (151.2, 92.2), turned to 180 degrees
- moved C14 37.4 mm to (151.3, 95.6), turned to 180 degrees
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Connections:
- R4 pad 1: Net-(U1-RUN) -> Net-(R4-Pad1)
- R4 pad 2: Net-(R4-Pad2) -> GND
- SW1 pad 1: unconnected-(SW1-Pad1) -> /~{USB_BOOT}
- SW1 pad 4: unconnected-(SW1-Pad4) -> GND
- SW2 pad 1: unconnected-(SW2-Pad1) -> Net-(U1-RUN)
- SW2 pad 2: Net-(R4-Pad2) -> Net-(U1-RUN)
- SW2 pad 3: GND -> Net-(R4-Pad1)
- SW2 pad 4: unconnected-(SW2-Pad4) -> Net-(R4-Pad1)
Routing:
- net GND: track 2.26 -> 34.0 mm, vias 5 -> 26
- net +3.3V: track 9.63 -> 36.5 mm, vias 0 -> 2
- net /QSPI_SS: track 0.00 -> 23.1 mm
- net /QSPI_SD1: track 0.00 -> 18.2 mm
- net +1V1: track 3.91 -> 21.8 mm, vias 2 -> 9
- net /USB_D-: track 0.00 -> 17.3 mm
- net /USB_D+: track 0.00 -> 17.3 mm
- net Net-(J2-Pin_2): track 0.00 -> 17.2 mm
- net Net-(J2-Pin_3): track 0.00 -> 15.7 mm
- net Net-(U1-RUN): track 0.00 -> 15.0 mm
- net /QSPI_SD2: track 0.00 -> 14.5 mm
- net /XIN: track 0.00 -> 14.4 mm
- net Net-(R4-Pad1): track 0.00 -> 11.7 mm
- net /~{USB_BOOT}: track 0.00 -> 11.6 mm
- net /QSPI_SD3: track 0.00 -> 10.8 mm
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- added copper zone on F.Cu, net VBUS

Commit message: Add part numbers
Parts:
- R4, R6: value 1K -> 1k
