File: rp2350_dev_board.kicad_sch (KiCad schematic)
At the start: 33 parts, among them J1 USB_B_Micro, J2 Conn_01x03_Socket, SW1 TS110426045, SW2 TS110426045, U1 RP2350A, U2 NCP1117-3.3_SOT223, U3 W25Q32JVSS, Y1 Crystal_GND24

Commit message: Minimal board complete
Parts:
- C2: value C -> 100n
- C6, C7: footprint Capacitor_SMD:C_0402_1005Metric -> rp2350:C_0402_1005Metric_small_pads
- R2: value 2K -> 1k
Connections:
- net GND: now also R4.2, SW1.4; no longer SW2.3
- net ~{USB_BOOT}: now also SW1.1
- net at SW2.1: now also SW2.2, U1.26 (RUN)
- net at SW2.4: now also R4.1, SW2.3
- no-connect marks 35 -> 31

Commit message: Add part numbers
Parts:
- R4, R6: value 1K -> 1k
Changed lines of the file:
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@@
 			)
 		)
-		(property "Value" "1K"
+		(property "Value" "1k"
 			(at 186.69 99.06 90)
 			(show_name no)
@@
 			)
 		)
-		(property "Value" "1K"
+		(property "Value" "1k"
 			(at 175.26 71.12 90)
 			(show_name no)
